Commit message: made changes, updated offsets to work with horizontal grasping also

File: neo_ur_moveit_config/srdf/mpo_700.srdf.xacro (robot description, xacro)
@@ -38,4 +38,12 @@
       <joint name="${prefix_value}wrist_2_joint" value="-1.6" />
       <joint name="${prefix_value}wrist_3_joint" value="-0.11" />
+    </group_state>
+    <group_state name="intermediate_pose" group="ur_manipulator">
+      <joint name="${prefix_value}elbow_joint" value="1.5" />
+      <joint name="${prefix_value}shoulder_lift_joint" value="-1.8" />
+      <joint name="${prefix_value}shoulder_pan_joint" value="2" />
+      <joint name="${prefix_value}wrist_1_joint" value="-1.6" />
+      <joint name="${prefix_value}wrist_2_joint" value="-1.5" />
+      <joint name="${prefix_value}wrist_3_joint" value="0" />
     </group_state>
     <!--DISABLE COLLISIONS: By default it is assumed that any link of the robot could potentially come into collision with any other link in the robot. This tag disables collision checking between a specified pair of links. -->

File: neo_ur_moveit_config/srdf/robotiq_2f_85.srdf.xacro (robot description, xacro)
@@ -18,8 +18,9 @@
     </group>
     <group_state name="open" group="gripper">
-      <joint name="robotiq_85_left_knuckle_joint" value="0.1" />
+      <joint name="robotiq_85_left_knuckle_joint" value="0.0" />
     </group_state>
     <group_state name="close" group="gripper">
-      <joint name="robotiq_85_left_knuckle_joint" value="0.2" />
+      <!-- gripper_closed_position from it's urdf -->
+      <joint name="robotiq_85_left_knuckle_joint" value="0.7929" />
     </group_state>
     <end_effector name="endeffector" group="gripper" parent_link="${prefix_value}wrist_3_link"/>
