Commit message: exec not working yet

File: neo_ur_moveit_config/srdf/robotiq_2f_85.srdf.xacro (robot description, xacro)
@@ -4,8 +4,19 @@
     A URDF file must exist for this robot as well, where the joints and the links that are referenced are defined
 -->
-<robot xmlns:xacro="http://www.ros.org/wiki/xacro" name="mpo_700">
+<robot xmlns:xacro="http://www.ros.org/wiki/xacro" name="2f_85">
   <xacro:arg name="prefix" default=""/>
   <xacro:property name="prefix_value" value="$(arg prefix)"/>
   <xacro:macro name="robotiq_2f_85">
+    <!-- EE group for MTC-->
+    <group name="gripper">
+      <joint name="robotiq_85_left_knuckle_joint"/>
+    </group>
+    <group_state name="open" group="gripper">
+      <joint name="robotiq_85_left_knuckle_joint" value="0.0" />
+    </group_state>
+    <group_state name="close" group="gripper">
+      <joint name="robotiq_85_left_knuckle_joint" value="0.8" />
+    </group_state>
+    <end_effector name="endeffector" group="gripper" parent_link="${prefix_value}wrist_3_link"/>
     <!--DISABLE COLLISIONS: By default it is assumed that any link of the robot could potentially come into collision with any other link in the robot. This tag disables collision checking between a specified pair of links. -->
     <disable_collisions link1="robotiq_85_base_link" link2="robotiq_85_left_finger_link" reason="Never"/>

Commit message: working planning version, have video

File: neo_ur_moveit_config/srdf/robotiq_2f_85.srdf.xacro (robot description, xacro)
@@ -8,4 +8,20 @@
   <xacro:property name="prefix_value" value="$(arg prefix)"/>
   <xacro:macro name="robotiq_2f_85">
+    <!-- EE group for MTC-->
+    <group name="gripper">
+      <link name="robotiq_85_base_link"/>
+      <link name="robotiq_85_left_finger_link"/>
+      <link name="robotiq_85_right_finger_link"/>
+      <link name="robotiq_85_left_finger_tip_link"/>
+      <link name="robotiq_85_right_finger_tip_link"/>
+      <joint name="robotiq_85_left_knuckle_joint"/>
+    </group>
+    <group_state name="open" group="gripper">
+      <joint name="robotiq_85_left_knuckle_joint" value="0.1" />
+    </group_state>
+    <group_state name="close" group="gripper">
+      <joint name="robotiq_85_left_knuckle_joint" value="0.33" />
+    </group_state>
+    <end_effector name="endeffector" group="gripper" parent_link="${prefix_value}wrist_3_link"/>
     <!--DISABLE COLLISIONS: By default it is assumed that any link of the robot could potentially come into collision with any other link in the robot. This tag disables collision checking between a specified pair of links. -->
     <disable_collisions link1="robotiq_85_base_link" link2="robotiq_85_left_finger_link" reason="Never"/>

Commit message: [WORKING]pick cube place cube pipeline working, with gz custom plugin service bridge also

File: neo_ur_moveit_config/srdf/robotiq_2f_85.srdf.xacro (robot description, xacro)
@@ -21,5 +21,5 @@
     </group_state>
     <group_state name="close" group="gripper">
-      <joint name="robotiq_85_left_knuckle_joint" value="0.33" />
+      <joint name="robotiq_85_left_knuckle_joint" value="0.25" />
     </group_state>
     <end_effector name="endeffector" group="gripper" parent_link="${prefix_value}wrist_3_link"/>

Commit message: [WORKING] can place single coke can

File: neo_ur_moveit_config/srdf/robotiq_2f_85.srdf.xacro (robot description, xacro)
@@ -21,5 +21,5 @@
     </group_state>
     <group_state name="close" group="gripper">
-      <joint name="robotiq_85_left_knuckle_joint" value="0.25" />
+      <joint name="robotiq_85_left_knuckle_joint" value="0.2" />
     </group_state>
     <end_effector name="endeffector" group="gripper" parent_link="${prefix_value}wrist_3_link"/>

Commit message: [WORKING]like a magic, the srdf gripper position groups were wrong, transformations now fixed

File: neo_ur_moveit_config/srdf/robotiq_2f_85.srdf.xacro (robot description, xacro)
@@ -17,10 +17,9 @@
       <joint name="robotiq_85_left_knuckle_joint"/>
     </group>
+    <group_state name="close" group="gripper">
+      <joint name="robotiq_85_left_knuckle_joint" value="0.2" />
+    </group_state>
     <group_state name="open" group="gripper">
       <joint name="robotiq_85_left_knuckle_joint" value="0.0" />
-    </group_state>
-    <group_state name="close" group="gripper">
-      <!-- gripper_closed_position from it's urdf -->
-      <joint name="robotiq_85_left_knuckle_joint" value="0.7929" />
     </group_state>
     <end_effector name="endeffector" group="gripper" parent_link="${prefix_value}wrist_3_link"/>

Commit message: not working im reverting to old branch since I created new pkg, saving this for any ref just in case

File: neo_ur_moveit_config/srdf/robotiq_2f_85.srdf.xacro (robot description, xacro)
@@ -18,8 +18,8 @@
     </group>
     <group_state name="close" group="gripper">
-      <joint name="robotiq_85_left_knuckle_joint" value="0.2" />
+      <joint name="robotiq_85_left_knuckle_joint" value="0.7929" />
     </group_state>
     <group_state name="open" group="gripper">
-      <joint name="robotiq_85_left_knuckle_joint" value="0.0" />
+      <joint name="robotiq_85_left_knuckle_joint" value="0.1" />
     </group_state>
     <end_effector name="endeffector" group="gripper" parent_link="${prefix_value}wrist_3_link"/>
